File: pcb/MacroHackClub.kicad_pcb (KiCad board)
At the start: 2 copper layers, 100 x 100 mm, 33 parts, among them J1 Conn_01x04_Pin, SW1 RotaryEncoder_Switch, SW2 SW_Push, SW3 SW_Push, SW4 SW_Push, SW5 SW_Push, SW6 SW_Push, SW7 SW_Push, U1 MOUDLE-SEEEDUINO-XIAO

Commit message: fixed issue
Routing:
- net Net-(D6-DOUT): track 71.1 -> 124.8 mm
- net Net-(D19-A): track 70.0 -> 74.6 mm
- net Net-(D21-A): track 81.8 -> 85.2 mm
- net Net-(U1-PA02_A0_D0): track 201.1 -> 203.7 mm
- net Net-(D17-A): track 61.1 -> 62.2 mm
- net Net-(D16-A): track 71.2 -> 72.0 mm
